Commit message: SISTEMA DE MEDICION

File: src/simulate/urdf/metodo_prueba.xacro (robot description, xacro)
@@ -6,5 +6,5 @@
       <origin xyz="0 0 0.003" rpy="0 0 0"/> <!-- Colocar el cubo en el suelo (0.075m de altura) -->
       <geometry>
-        <box size="0.25 0.25 0.06"/> <!-- Tamaño del cubo: 15cm x 15cm x 15cm -->
+        <box size="0.15 0.15 0.06"/> <!-- Tamaño del cubo: 15cm x 15cm x 15cm -->
       </geometry>
       <material name="texture_material">

File: src/simulate/urdf/sawyer_base.urdf.xacro (robot description, xacro)
@@ -557,5 +557,5 @@
   <!-- Joint entre la mano y la esfera -->
   <joint name="right_hand_to_sphere_joint" type="fixed">
-    <origin rpy="1.573 0.3 3.14" xyz="0 0 0.05"/> <!-- Colocamos la esfera a 5 cm de la mano -->
+    <origin rpy="0 0 0" xyz="0 0 0.05"/> <!-- Colocamos la esfera a 5 cm de la mano -->
     <parent link="right_hand"/> <!-- La esfera está conectada a la mano -->
     <child link="right_hand_sphere"/> <!-- La esfera como hijo -->

Commit message: Data

File: src/simulate/urdf/metodo_prueba.xacro (robot description, xacro)
@@ -6,5 +6,5 @@
       <origin xyz="0 0 0.003" rpy="0 0 0"/> <!-- Colocar el cubo en el suelo (0.075m de altura) -->
       <geometry>
-        <box size="0.15 0.15 0.06"/> <!-- Tamaño del cubo: 15cm x 15cm x 15cm -->
+        <box size="0.1 0.1 0.06"/> <!-- Tamaño del cubo: 15cm x 15cm x 15cm -->
       </geometry>
       <material name="texture_material">

Commit message: dATA

File: src/simulate/urdf/metodo_prueba.xacro (robot description, xacro)
@@ -4,7 +4,7 @@
   <link name="small_cube_link">
     <visual>
-      <origin xyz="0 0 0.003" rpy="0 0 0"/> <!-- Colocar el cubo en el suelo (0.075m de altura) -->
+      <origin xyz="0 0 -0.015" rpy="0 0 0"/> <!-- Colocar el cubo en el suelo (0.075m de altura) -->
       <geometry>
-        <box size="0.1 0.1 0.06"/> <!-- Tamaño del cubo: 15cm x 15cm x 15cm -->
+        <box size="0.1 0.1 0.03"/> <!-- Tamaño del cubo: 15cm x 15cm x 15cm -->
       </geometry>
       <material name="texture_material">
